File: psrtest.sch (KiCad schematic (older format))
At the start: 1 part, among them U1 IS66WVE4M16EBLL-70BLI

Commit message: Initial fanout.
Parts:
- added J1, J2, J3, J4: Conn_01x12, Pin_Headers:Pin_Header_Straight_1x12_Pitch2.54mm, symbol Conn_01x12
Connections:
- net labels added: A0, A1, A10, A11, A12, A13, A14, A15, A16, A17, A18, A19, A2, A20, A21, A3, A4, A5, A6, A7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
- wire segments 0 -> 112
Other:
- moved on the sheet: U1
